File: Hardware/lowspeed-modem/modem-breakout.brd (EAGLE design)
At the start: 79.2 x 42.6 mm, 5 parts, among them J1 8468-11B1-RK-TP, J2 RJ11-2L-B

Commit message: nerp
Parts:
- added C3, C4: 4.7uf, rcl:C0805
- added JP1: (no value), pinhead:1X02
- added JP2: (no value), pinhead:1X12
- added U1: AP2111H-3.3, AP2111H-3.3TRG1:SOT-223_DIO-M
- J2: value RJ11-2L-B -> 1-1705950-2
Connections:
- new net +5V: C3.1, JP2.12, U1.3
- net !CTS: now also JP2.9
- net !DCD: now also JP2.11
- net !DSR: now also JP2.7
- net !DTR: now also JP2.5
- net !INT: now also JP2.2
- net !RESET: now also JP2.10
- net !RI: now also JP2.4
- net !RST: now also JP2.8
- net !RXD: now also JP2.6
- net !TXD: now also JP2.3
- net GND: now also C3.2, C4.2, JP1.1, JP2.1, U1.1
- net SPKR: now also JP1.2
- net VCC: now also C4.1, U1.2
Routing:
- net +5V: track 0.00 -> 64.3 mm
- net VCC: track 0.00 -> 57.4 mm, vias 0 -> 1
- net TIP: track 0.00 -> 22.5 mm
- net !RESET: track 0.00 -> 20.2 mm
- net !DCD: track 0.00 -> 19.9 mm
- net !RST: track 0.00 -> 18.8 mm
- net SPKR: track 0.00 -> 18.0 mm
- net !RXD: track 0.00 -> 17.8 mm
- net !RI: track 0.00 -> 17.4 mm
- net !INT: track 0.00 -> 17.4 mm
- net RING: track 0.00 -> 16.9 mm
- net !CTS: track 0.00 -> 16.3 mm
- net !DSR: track 0.00 -> 15.2 mm
- net !TXD: track 0.00 -> 14.8 mm
- net !DTR: track 0.00 -> 14.3 mm
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- added copper zone on layer 1, net GND
- added copper zone on layer 16, net GND
Other:
- board size 79.2 x 42.6 mm -> 71.1 x 42.6 mm
- board text added: "!CTS"
- board text added: "!DCD"
- board text added: "!DSR"
- board text added: "!DTR"
- board text added: "!INT"
- board text added: "!RESET"
- board text added: "!RI"
- board text added: "!RST"
- board text added: "!RXD"
- board text added: "!TXD"
- board text added: "+5"
- board text added: "GND"
- board text added: "MJM 2022"
- board text added: "SPKR"
- board text added: "Single Chip Breakout"
- board text added: "Smallest World-Wide 2400 BPS Modem"
- board text added: "XE2420G"
- board text added: "XECOM"

Commit message: update
Parts:
- J2: device con-tycoelectronics:RJ11-NO_SHIELD -> con-tycoelectronics_copy:RJ11-NO_SHIELD
Changed lines of the file:
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@@
 </layers>
 <board>
-<fusionsync huburn="a.YnVzaW5lc3M6bWljcm9jb21jb3Jw" projecturn="a.YnVzaW5lc3M6bWljcm9jb21jb3JwI0QyMDIxMDYxMDQxOTQ4MzU4MQ" f3durn="urn:adsk.wipprod:dm.lineage:LzuZvWWlQPyJhGtXXWPxQw" pcbguid="" lastpulledtime="" lastsyncedchangeguid="" latestrevisionid="af75e047-1152-4c6d-9cae-9e98044a9383" lastsyncedrevisionid="af75e047-1152-4c6d-9cae-9e98044a9383" lastboardhashguid="61031957-6967-2afc-d451-abf78d08c86a" lastpushedtime="2022-01-01T23:28:51Z" linktopcb3d="true"/>
+<fusionsync huburn="a.YnVzaW5lc3M6bWljcm9jb21jb3Jw" projecturn="a.YnVzaW5lc3M6bWljcm9jb21jb3JwI0QyMDIxMDYxMDQxOTQ4MzU4MQ" f3durn="urn:adsk.wipprod:dm.lineage:LzuZvWWlQPyJhGtXXWPxQw" pcbguid="" lastpulledtime="" lastsyncedchangeguid="" latestrevisionid="3d90f0ff-372a-4452-86a0-9c1ca5f5b2b4" lastsyncedrevisionid="3d90f0ff-372a-4452-86a0-9c1ca5f5b2b4" lastboardhashguid="5c6f4c84-b72e-239e-59ac-1270da0e2af2" lastpushedtime="2022-01-02T00:11:29Z" linktopcb3d="true"/>
 <plain>
 <wire x1="0" y1="0" x2="71.1" y2="0" width="0" layer="20"/>
@@
 </autorouter>
 <elements>
-<element name="J1" library="8468-11B1-RK-TP" library_urn="urn:adsk.eagle:library:33322605" package="3M_8468-11B1-RK-TP" package3d_urn="urn:adsk.eagle:package:33322608/1" value="8468-11B1-RK-TP" x="29.464" y="17.526" smashed="yes" rot="R90">
+<element name="J1" library="8468-11B1-RK-TP" library_urn="urn:adsk.eagle:library:33322605" package="3M_8468-11B1-RK-TP" package3d_urn="urn:adsk.eagle:package:33322608/2" value="8468-11B1-RK-TP" x="29.464" y="17.526" smashed="yes" rot="R90">
 <attribute name="AVAILABILITY" value="In Stock" x="48.514" y="46.736" size="1.778" layer="27" rot="R90" display="off"/>
 <attribute name="DESCRIPTION" value=" 68 (4 x 17) Pos PLCC Socket Tin Through Hole " x="48.514" y="46.736" size="1.778" layer="27" rot="R90" display="off"/>
@@
 <attribute name="NAME" x="59.69" y="21.844" size="0.8128" layer="25" font="vector" ratio="16"/>
 </element>
-<element name="J2" library="con-tycoelectronics" library_urn="urn:adsk.eagle:library:193" package="RJ11-NO_SHIELD" package3d_urn="urn:adsk.eagle:package:10656/1" value="1-1705950-2" x="60.706" y="5.588" smashed="yes">
+<element name="J2" library="con-tycoelectronics_copy" library_urn="urn:adsk.eagle:library:33324054" package="RJ11-NO_SHIELD" package3d_urn="urn:adsk.eagle:package:33324049/2" value="1-1705950-2" x="60.706" y="5.588" smashed="yes">
 <attribute name="MF" value="TYCO ELECTRONICS" x="60.706" y="5.588" size="1.778" layer="27" display="off"/>
 <attribute name="MPN" value="RJ11-2L-B" x="60.706" y="5.588" size="1.778" layer="27" display="off"/>
@@
 <attribute name="POPULARITY" value="0" x="60.706" y="5.588" size="1.778" layer="27" display="off"/>
 </element>
-<element name="U1" library="AP2111H-3.3TRG1" library_urn="urn:adsk.eagle:library:29764339" package="SOT-223_DIO-M" package3d_urn="urn:adsk.eagle:package:29764344/2" value="AP2111H-3.3" x="58.166" y="29.464" smashed="yes" rot="R90">
+<element name="U1" library="AP2111H-3.3TRG1" library_urn="urn:adsk.eagle:library:29764339" package="SOT-223_DIO-M" package3d_urn="urn:adsk.eagle:package:29764344/3" value="AP2111H-3.3" x="58.166" y="29.464" smashed="yes" rot="R90">
 <attribute name="BUILT_BY" value="EMA_UL_Team" x="58.166" y="29.464" size="1.778" layer="27" rot="R90" display="off"/>
 <attribute name="MANUFACTURER_PART_NUMBER" value="AP2111H-3.3TRG1" x="58.166" y="29.464" size="1.778" layer="27" rot="R90" display="off"/>
