File: Hardware/lowspeed-modem/modem-breakout.sch (EAGLE design)
At the start: 5 parts, among them J1 8468-11B1-RK-TP, J2 RJ11-2L-B

Commit message: nerp
Parts:
- added C3, C4: 4.7uf, rcl:C-EUC0805
- added JP1: (no value), pinhead:PINHD-1X2
- added JP2: (no value), pinhead:PINHD-1X12
- added U1: AP2111H-3.3, AP2111H-3.3TRG1:AP2111H-3.3TRG1SOT-223_DIO-M
- J2: value RJ11-2L-B -> 1-1705950-2
Connections:
- new net +5V: C3.1, JP2.12, U1.VIN
- net !CTS: now also JP2.9
- net !DCD: now also JP2.11
- net !DSR: now also JP2.7
- net !DTR: now also JP2.5
- net !INT: now also JP2.2
- net !RESET: now also JP2.10
- net !RI: now also JP2.4
- net !RST: now also JP2.8
- net !RXD: now also JP2.6
- net !TXD: now also JP2.3
- net GND: now also C3.2, C4.2, JP1.1, JP2.1, U1.GND
- net SPKR: now also JP1.2
- net VCC: now also C4.1, U1.VOUT

Commit message: update
Parts:
- J2: device con-tycoelectronics:RJ11-2L-B -> con-tycoelectronics_copy:RJ11-2L-B
Changed lines of the file:
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@@
 </classes>
 <parts>
-<part name="J1" library="8468-11B1-RK-TP" library_urn="urn:adsk.eagle:library:33322605" deviceset="8468-11B1-RK-TP" device="" package3d_urn="urn:adsk.eagle:package:33322608/1"/>
+<part name="J1" library="8468-11B1-RK-TP" library_urn="urn:adsk.eagle:library:33322605" deviceset="8468-11B1-RK-TP" device="" package3d_urn="urn:adsk.eagle:package:33322608/2"/>
 <part name="FRAME1" library="frames" library_urn="urn:adsk.eagle:library:229" deviceset="A4L-LOC" device=""/>
 <part name="C1" library="rcl" library_urn="urn:adsk.eagle:library:334" deviceset="C-EU" device="075-052X106" package3d_urn="urn:adsk.eagle:package:23650/1" value="S471K33Y5PR63K7R"/>
@@
 <part name="GND2" library="supply1" library_urn="urn:adsk.eagle:library:371" deviceset="GND" device=""/>
 <part name="PTC1" library="TR600-150F-EX" library_urn="urn:adsk.eagle:library:33322685" deviceset="TR600-150F-EX" device="" package3d_urn="urn:adsk.eagle:package:33322688/2" value="TR600-150F-EX"/>
-<part name="J2" library="con-tycoelectronics" library_urn="urn:adsk.eagle:library:193" deviceset="RJ11" device="" package3d_urn="urn:adsk.eagle:package:10656/1" technology="-2L-B" value="1-1705950-2"/>
-<part name="U1" library="AP2111H-3.3TRG1" library_urn="urn:adsk.eagle:library:29764339" deviceset="AP2111H-3.3TRG1" device="SOT-223_DIO-M" package3d_urn="urn:adsk.eagle:package:29764344/2" value="AP2111H-3.3"/>
+<part name="J2" library="con-tycoelectronics_copy" library_urn="urn:adsk.eagle:library:33324054" deviceset="RJ11" device="" package3d_urn="urn:adsk.eagle:package:33324049/2" technology="-2L-B" value="1-1705950-2"/>
+<part name="U1" library="AP2111H-3.3TRG1" library_urn="urn:adsk.eagle:library:29764339" deviceset="AP2111H-3.3TRG1" device="SOT-223_DIO-M" package3d_urn="urn:adsk.eagle:package:29764344/3" value="AP2111H-3.3"/>
 <part name="GND3" library="supply1" library_urn="urn:adsk.eagle:library:371" deviceset="GND" device=""/>
 <part name="C3" library="rcl" library_urn="urn:adsk.eagle:library:334" deviceset="C-EU" device="C0805" package3d_urn="urn:adsk.eagle:package:23617/2" value="4.7uf"/>
